File: link101_carrier/link101_carrier.kicad_pcb (KiCad board)
At the start: 4 copper layers, 91.1 x 64.4 mm, 45 parts, among them CN1 5264-4P ZZMS, CN2 5264-3P ZZMS, CN5 MKDS1/3-3.5, CN6 MKDS1/3-3.5, CN7 5264-3P ZZMS, CN8 XY-SM04B-GHS-TB, CN9 XT30(2+2)PB-M.G.B, J1 Conn_01x03_Pin, J10 Conn_02x06_Counter_Clockwise, J11 Conn_02x06_Counter_Clockwise, J12 Conn_02x06_Counter_Clockwise, J13 Conn_01x12_Socket, J19 Screw_Terminal_01x02, J20 Screw_Terminal_01x02, J21 Conn_01x15_Pin, J22 Conn_01x15_Pin, J3 Qwiic_Vertical, J4 Conn_01x03_Pin, J5 Conn_01x04_Socket, J6 Conn_01x03_Pin, J7 Conn_01x15_Pin, J8 Conn_01x04_Socket, J9 Conn_01x04_Socket, U1 link101_Module, U10 XL-1010RGBC-WS2812B, U11 XL-1010RGBC-WS2812B, U13 XL-1010RGBC-WS2812B, U3 LSM6DSOX, U5 MMC5983MA, U6 LMR16006YDDCR, U7 XL-1010RGBC-WS2812B, U8 XL-1010RGBC-WS2812B, U9 XL-1010RGBC-WS2812B

Commit message: added pcb files
Parts:
- removed L4: SMNR5040-150MT, easyeda2kicad:IND-SMD_L5.0-W5.0_SMNR5040
- added JP1: SolderJumper_2_Open, Jumper:SolderJumper-2_P1.3mm_Open_RoundedPad1.0x1.5mm, F.Cu at (205.0, 123.0)
- added JP2: SolderJumper_2_Open, Jumper:SolderJumper-2_P1.3mm_Open_RoundedPad1.0x1.5mm, F.Cu at (205.0, 120.0)
- added L1: L, Inductor_SMD:L_Cenker_CKCS5040, F.Cu at (209.0, 102.3)
- added RFB1: 54.9k, Resistor_SMD:R_0603_1608Metric, F.Cu at (205.0, 104.0)
- added RFB2: 10k, Resistor_SMD:R_0603_1608Metric, F.Cu at (203.0, 104.0)
- moved U1 237.4 mm to (220.8, 88.2), turned to -90 degrees
- moved REN1 11.6 mm to (198.5, 102.2), turned to 0 degrees
- moved C9 9.00 mm to (199.0, 104.4)
- moved U6 8.22 mm to (199.5, 99.2), turned to 180 degrees
- moved C2 6.07 mm to (214.0, 102.5), turned to 90 degrees
- moved D2 5.00 mm to (214.0, 110.3)
- moved D3 5.00 mm to (209.0, 110.3)
- moved D5V1 1.82 mm to (208.1, 96.8)
- moved CBOOT_5V1 1.32 mm to (203.5, 100.2), turned to -90 degrees
Connections:
- U3 pad 4: /INT_IMU -> Net-(JP1-B)
- U5 pad 15: /INT_MAG -> Net-(JP2-A)
- U6 pad 3: /VBUS -> Net-(U6-FB)
Routing:
- net /PWR: track 0.00 -> 81.1 mm, vias 16 -> 96
- net /RS485_B_1: track 75.6 -> 112.4 mm
- net /RS485_A_1: track 73.2 -> 100.0 mm
- net /INT_IMU: track 37.9 -> 17.6 mm, vias 2 -> 1
- net /VSERVO: track 0.00 -> 18.4 mm, vias 30 -> 289
- net Net-(JP1-B): track 0.00 -> 17.5 mm, vias 0 -> 2
- net /VIN: track 6.59 -> 23.5 mm, vias 2 -> 0
- net /INT_MAG: track 33.4 -> 17.8 mm, vias 2 -> 1
- net /SCL: track 71.0 -> 83.7 mm, vias 1 -> 3
- net Net-(JP2-A): track 0.00 -> 12.6 mm, vias 0 -> 1
- net GND: track 69.9 -> 58.4 mm
- net Net-(U6-FB): track 0.00 -> 10.8 mm, vias 0 -> 2
- net /CAN_H: track 92.8 -> 102.8 mm
- net /VBUS: track 50.1 -> 59.0 mm
- net Net-(D5V1-K): track 5.75 -> 0.00 mm
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- added copper zone on In1.Cu, net /PWR
- added copper zone on In2.Cu, net /PWR
- added copper zone on B.Cu, net GND
- added copper zone on F.Cu, net GND
- added copper zone on In1.Cu, net GND
- added copper zone on In2.Cu, net GND
- added copper zone on F.Cu, net Net-(D5V1-K)
Other:
- board text added: "{ "ViaStitching": "0.2", "stitch_zone_0": { "HSpacing": "1.25", "VSpacing": "1.25", "HOffset": "0", "VOffset": "0", "Clearance": "0", "Randomize": false } }"
- board text added: "{ "ViaStitching": "0.2", "stitch_zone_0": { "HSpacing": "1.5", "VSpacing": "1.5", "HOffset": "0", "VOffset": "0", "Clearance": "0", "Randomize": false } }"
- board text added: "{ "ViaStitching": "0.2", "stitch_zone_0": { "HSpacing": "2", "VSpacing": "2", "HOffset": "0", "VOffset": "0", "Clearance": "0", "Randomize": false } }"
- board text added: "{ "ViaStitching": "0.2", "stitch_zone_0": { "HSpacing": "2.5", "VSpacing": "2.5", "HOffset": "0", "VOffset": "0", "Clearance": "0", "Randomize": false } }"
