File: link101_carrier/link101_carrier.kicad_sch (KiCad schematic)
At the start: 47 parts, among them CN1 5264-4P ZZMS, CN2 5264-3P ZZMS, CN5 MKDS1/3-3.5, CN6 MKDS1/3-3.5, CN7 5264-3P ZZMS, CN8 XY-SM04B-GHS-TB, CN9 XT30(2+2)PB-M.G.B, J1 Conn_01x03_Pin, J10 Conn_02x06_Counter_Clockwise, J11 Conn_02x06_Counter_Clockwise, J12 Conn_02x06_Counter_Clockwise, J13 Conn_01x12_Socket, J19 Screw_Terminal_01x02, J20 Screw_Terminal_01x02, J21 Conn_01x15_Pin, J22 Conn_01x15_Pin, J3 Qwiic_Vertical, J4 Conn_01x03_Pin, J5 Conn_01x04_Socket, J6 Conn_01x03_Pin, J7 Conn_01x15_Pin, J8 Conn_01x04_Socket, J9 Conn_01x04_Socket, U1 link101_Module, U10 XL-1010RGBC-WS2812B, U11 XL-1010RGBC-WS2812B, U13 XL-1010RGBC-WS2812B, U3 LSM6DSOX, U5 MMC5983MA, U6 LMR16006YDDCR, U7 XL-1010RGBC-WS2812B, U8 XL-1010RGBC-WS2812B, U9 XL-1010RGBC-WS2812B

Commit message: added pcb files
Parts:
- removed L4: SMNR5040-150MT, easyeda2kicad:IND-SMD_L5.0-W5.0_SMNR5040, symbol easyeda2kicad_1:SMNR5040-150MT
- added L1: L, Inductor_SMD:L_Cenker_CKCS5040, symbol Device:L
- added RFB1: 54.9k, Resistor_SMD:R_0603_1608Metric, symbol Device:R
- added RFB2: 10k, Resistor_SMD:R_0603_1608Metric, symbol Device:R
- JP1, JP2: footprint (none) -> Jumper:SolderJumper-2_P1.3mm_Open_RoundedPad1.0x1.5mm
Connections:
- net GND: now also RFB2.1
- net INT_MAG: now also JP2.2 (B)
- net VBUS: now also L1.2, RFB1.2; no longer U6.3 (FB)
- net at CBOOT_5V1.2, D5V1.1 (K), U6.6 (SW): now also L1.1
- new net: RFB1.1, RFB2.2, U6.3 (FB)
Other:
- moved on the sheet: J8, J9
